File: pcbs/main_board/main_board.kicad_sch (KiCad schematic)
At the start: 6 parts, among them J3 LED strip, J4 Motor, P1 USB/STEPUP, U1 mini_esp32

Commit message: Add connectors
Parts:
- J3: footprint (none) -> Connector_JST:JST_XH_S3B-XH-A-1_1x03_P2.50mm_Horizontal; Manufacturer Part Number (none) -> S3B-XH-A-E(LF)(SN); Supplier (none) -> Mouser; Supplier Part Number (none) -> 306-S3BXHAELFSN
- J4: footprint (none) -> Connector_JST:JST_XH_S2B-XH-A-1_1x02_P2.50mm_Horizontal; Manufacturer Part Number (none) -> S2B-XH-A-BK(LF)(SN); Supplier (none) -> Mouser; Supplier Part Number (none) -> 306-S2BXHABKLFSN
- P1: footprint Connector_PinHeader_2.54mm:PinHeader_1x03_P2.54mm_Vertical -> Connector_PinHeader_2.54mm:PinHeader_1x03_P2.54mm_Horizontal; Manufacturer Part Number (none) -> LA217003A; Supplier (none) -> LaskaKit; Supplier Part Number (none) -> LA217003A
- U1: Manufacturer Part Number (none) -> LA100089
Connections:
- net B_STATUS: now reaches U1.6 (IO_26/D0)
Other:
- sheet Power distribution ports: added STATUS; removed none
- note added: "TODO: - U datové linky LED pásku je k zamyšlení level shifter 3.3V -> 5V - Přidat nějaké signal LED"
- note removed: "TODO: - U datové linky LED pásku je k zamyšlení level shifter 3.3V -> 5V - Vybrat konektory na desku, asi jst-xh? - Přidat nějaké signal LED"
Changed lines of the file:
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@@
 	(generator_version "9.0")
 	(paper "A4")
-	(text "TODO:\n- U datové linky LED pásku je k zamyšlení level shifter 3.3V -> 5V\n- Vybrat konektory na desku, asi jst-xh?\n- Přidat nějaké signal LED\n"
+	(text "TODO:\n- U datové linky LED pásku je k zamyšlení level shifter 3.3V -> 5V\n- Přidat nějaké signal LED\n"
 		(exclude_from_sim no)
 		(at 180.848 141.732 0)
@@
 	(wire
 		(pts
+			(xy 133.35 100.33) (xy 135.89 100.33)
+		)
+		(stroke
+			(width 0)
+			(type default)
+		)
+	)
+	(wire
+		(pts
 			(xy 121.92 34.29) (xy 121.92 46.99)
 		)
@@
 	(wire
 		(pts
+			(xy 39.37 24.13) (xy 43.18 24.13)
+		)
+		(stroke
+			(width 0)
+			(type default)
+		)
+	)
+	(wire
+		(pts
 			(xy 121.92 57.15) (xy 121.92 49.53)
 		)
@@
 		)
 	)
+	(hierarchical_label "B_STATUS"
+		(shape input)
+		(at 133.35 100.33 180)
+		(effects
+			(font
+				(size 1.27 1.27)
+			)
+			(justify right)
+		)
+	)
 	(hierarchical_label "M_IPROP"
 		(shape input)
@@
 		)
 	)
+	(hierarchical_label "B_STATUS"
+		(shape output)
+		(at 43.18 24.13 0)
+		(effects
+			(font
+				(size 1.27 1.27)
+			)
+			(justify left)
+		)
+	)
 	(hierarchical_label "M_PWM"
 		(shape input)
@@
 			)
 		)
-		(property "Footprint" ""
+		(property "Footprint" "Connector_JST:JST_XH_S3B-XH-A-1_1x03_P2.50mm_Horizontal"
 			(at 86.36 34.29 0)
 			(effects
@@
 			)
 		)
-		(property "Datasheet" "~"
+		(property "Datasheet" "https://cz.mouser.com/datasheet/3/1070/1/eXH.pdf"
 			(at 86.36 34.29 0)
 			(effects
@@
 			)
 		)
-		(property "Description" "Generic screw terminal, single row, 01x03, script generated (kicad-library-utils/schlib/autogen/connector/)"
+		(property "Description" "JST XH 3 pin, zásuvka, boční"
+			(at 86.36 34.29 0)
+			(effects
+				(font
+					(size 1.27 1.27)
+				)
+				(hide yes)
+			)
+		)
+		(property "Manufacturer Part Number" "S3B-XH-A-E(LF)(SN)"
+			(at 86.36 34.29 0)
+			(effects
+				(font
+					(size 1.27 1.27)
+				)
+				(hide yes)
+			)
+		)
+		(property "Supplier" "Mouser"
+			(at 86.36 34.29 0)
+			(effects
+				(font
+					(size 1.27 1.27)
+				)
+				(hide yes)
+			)
+		)
+		(property "Supplier Part Number" "306-S3BXHAELFSN"
 			(at 86.36 34.29 0)
 			(effects
@@
 			)
 		)
-		(property "Footprint" "Connector_PinHeader_2.54mm:PinHeader_1x03_P2.54mm_Vertical"
+		(property "Footprint" "Connector_PinHeader_2.54mm:PinHeader_1x03_P2.54mm_Horizontal"
 			(at 165.1 31.75 0)
 			(effects
@@
 			)
 		)
-		(property "Description" "Jumper"
+		(property "Description" "Kolíková lišta"
 			(at 165.1 31.75 0)
 			(effects
@@
 			)
 		)
+		(property "Manufacturer Part Number" "LA217003A"
+			(at 165.1 31.75 90)
+			(effects
+				(font
+					(size 1.27 1.27)
+				)
+				(hide yes)
+			)
+		)
+		(property "Supplier" "LaskaKit"
+			(at 165.1 31.75 90)
+			(effects
+				(font
+					(size 1.27 1.27)
+				)
+				(hide yes)
+			)
+		)
+		(property "Supplier Part Number" "LA217003A"
+			(at 165.1 31.75 90)
+			(effects
+				(font
+					(size 1.27 1.27)
+				)
+				(hide yes)
+			)
+		)
 		(pin "2"
 		)
@@
 			)
 		)
-		(property "Footprint" ""
+		(property "Footprint" "Connector_JST:JST_XH_S2B-XH-A-1_1x02_P2.50mm_Horizontal"
 			(at 251.46 31.75 0)
 			(effects
@@
 			)
 		)
-		(property "Datasheet" "~"
+		(property "Datasheet" "https://cz.mouser.com/datasheet/3/1070/1/eXH.pdf"
 			(at 251.46 31.75 0)
 			(effects
@@
 			)
 		)
-		(property "Description" "Generic screw terminal, single row, 01x02, script generated (kicad-library-utils/schlib/autogen/connector/)"
+		(property "Description" "JST XH 2 pin, zásuvka, boční"
+			(at 251.46 31.75 0)
+			(effects
+				(font
+					(size 1.27 1.27)
+				)
+				(hide yes)
+			)
+		)
+		(property "Manufacturer Part Number" "S2B-XH-A-BK(LF)(SN)"
+			(at 251.46 31.75 0)
+			(effects
+				(font
+					(size 1.27 1.27)
+				)
+				(hide yes)
+			)
+		)
+		(property "Supplier" "Mouser"
+			(at 251.46 31.75 0)
+			(effects
+				(font
+					(size 1.27 1.27)
+				)
+				(hide yes)
+			)
+		)
+		(property "Supplier Part Number" "306-S2BXHABKLFSN"
 			(at 251.46 31.75 0)
 			(effects
@@
 			)
 		)
-		(property "Manufacturer Part Number" "~"
+		(property "Manufacturer Part Number" "LA100089"
 			(at 148.59 39.37 0)
 			(effects
@@
 			)
 		)
+		(pin "STATUS" output
+			(at 39.37 24.13 0)
+			(effects
+				(font
+					(size 1.27 1.27)
+				)
+				(justify right)
+			)
+		)
