File: pcbs/main_board/untitled.kicad_sch (KiCad schematic)
At the start: 4 parts, among them U9 TXU0101

Commit message: Main board final update
Other:
- company: (none) -> Brno Mars Rover
- title: (none) -> Main board - MyMachine LED cap
Changed lines of the file:
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@@
 	(generator "eeschema")
 	(generator_version "9.0")
-	(paper "A5")
+	(paper "A4")
+	(title_block
+		(title "Main board - MyMachine LED cap")
+		(date "2026-01-20")
+		(company "Brno Mars Rover")
+	)
 	(junction
 		(at 118.11 63.5)

Commit message: changed footprint of level shifter
Parts:
- U9: footprint Package_TO_SOT_SMD:SOT-23-6_Handsoldering -> Package_TO_SOT_SMD:SOT-363_SC-70-6_Handsoldering; Manufacturer Part Number TXU0101DBVR -> TXU0101DCKR; Supplier Part Number 595-TXU0101DBVR -> 595-TXU0101DCKR
Changed lines of the file:
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@@
 			)
 		)
-		(property "Footprint" "Package_TO_SOT_SMD:SOT-23-6_Handsoldering"
+		(property "Footprint" "Package_TO_SOT_SMD:SOT-363_SC-70-6_Handsoldering"
 			(at 105.41 66.04 0)
 			(effects
@@
 			)
 		)
-		(property "Manufacturer Part Number" "TXU0101DBVR"
+		(property "Manufacturer Part Number" "TXU0101DCKR"
 			(at 105.41 66.04 0)
 			(effects
@@
 			)
 		)
-		(property "Supplier Part Number" "595-TXU0101DBVR"
+		(property "Supplier Part Number" "595-TXU0101DCKR"
 			(at 105.41 66.04 0)
 			(effects
