File: pcbs/main_board/main_board.kicad_pcb (KiCad board)
At the start: 2 copper layers, 70 x 61.2 mm, 56 parts, among them J1 BAT1, J2 BAT2, J3 LED strip, J4 Motor, Q1 NMOS, Q2 NMOS, SW1 Power switch, U1 mini_esp32, U10 LM74610QDGKRQ1, U11 LM74610QDGKRQ1, U2 ADXL345, U3 DRV8873HPWPRQ1, U4 Display, U5 Step-up, U6 TPS22917LDBV, U8 ST1L08, U9 TXU0101

Commit message: Main_board pcb v0.0
Parts:
- added G***: LOGO, LOGO, F.Cu at (46.2, 46.9)
- added G***: LOGO, LOGO, F.Cu at (54.0, 33.6)
- moved C16 9.66 mm to (95.5, 68.4), turned to 180 degrees
- moved F1 8.80 mm to (79.7, 68.7), turned to 180 degrees
- moved GND2 3.50 mm to (57.5, 40.6)
- moved GND1 3.48 mm to (57.5, 40.6)
- moved D4 0.09 mm to (32.1, 50.2)
- moved D2 0.07 mm to (32.1, 43.1)
- moved D1 0.07 mm to (32.1, 46.7)
Routing:
- net Net-(SW1A-A): track 47.8 -> 38.6 mm
- net Net-(U10-VCAPH): track 2.48 -> 9.60 mm
- net +5V: track 37.3 -> 44.0 mm
- net GND: track 352.2 -> 358.8 mm, vias 34 -> 33
- net Net-(U10-CATHODE): track 28.0 -> 33.1 mm
- net Net-(U10-VCAPL): track 6.87 -> 2.58 mm
Other:
- board size 70 x 61.2 mm -> 70 x 59.7 mm
- board text added: "3V3"
- board text added: "5V"
- board text added: "BAT"
- board text added: "BAT1"
- board text added: "BAT2"
- board text added: "DISPLAY"
- board text added: "Developed by:"
- board text added: "GND"
- board text added: "LED STRIP"
- board text added: "MOTOR"
- board text added: "POWER SWITCH"
- board text added: "v0.0 main_board"
- board text removed: "Foto boxu do kterého se PCB vloží (pro aktuální viz. Fusion projekt)"
- board text removed: "NOTES: - Rozměry PCB převzaty z modelu ve Fusionu - navrhl jsem umístění ESP, je potřeba ho umístit někam, kam se snadno vejde USB kabel, takže se klidně může přemístit, ale je třeba na to myslet - Když na to tak koukám, tak se vše pravděpodobně nevejde na jednu stranu, oboustrané PCB nevadí, jen by bylo vhodné dát na stranu FRONT konektory. - Co se týče konektorů obecně myslet na to, že za hrani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"
