File: pcbs/main_board/power_distribution.kicad_sch (KiCad schematic)
At the start: 22 parts, among them J1 BAT1, J2 BAT2, Q1 NMOS, Q2 NMOS, SW1 Power switch, U10 LM74610QDGKRQ1, U11 LM74610QDGKRQ1, U5 Step-up, U8 ST1L08

Commit message: Fix bom errors - main board
Parts:
- C16, C17: Supplier Part Number 603-CC603KRX7R9BB103 -> 80-C0603C104M5R
Changed lines of the file:
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@@
 			)
 		)
-		(property "Supplier Part Number" "603-CC603KRX7R9BB103"
+		(property "Supplier Part Number" "80-C0603C104M5R"
 			(at 50.8 57.15 0)
 			(effects
@@
 			)
 		)
-		(property "Supplier Part Number" "603-CC603KRX7R9BB103"
+		(property "Supplier Part Number" "80-C0603C104M5R"
 			(at 50.8 115.57 0)
 			(effects
